Commit message: feat(VSS): change robot parameters and reward weights

File: envs/vss_robot.urdf (robot description, URDF)
Before this commit: robot vss, 5 links, 4 joints
Links:
- link body: mass 0.4 -> 0.296; geometry collision box size=0.08 0.08 0.056; visual box size=0.08 0.08 0.056
- link leftWheel: mass 0.02 -> 0.021; geometry collision sphere radius=0.026; visual cylinder length=0.0025 radius=0.026
- link rightWheel: mass 0.02 -> 0.021; geometry collision sphere radius=0.026; visual cylinder length=0.0025 radius=0.026
Joints:
- joint body_leftWheel: limit effort=0.1 velocity=150.0 -> effort=0.0211 velocity=133.0
- joint body_rightWheel: limit effort=0.1 velocity=150.0 -> effort=0.0211 velocity=133.0
